File: hardware/MCC20.sch (KiCad schematic (older format))
At the start: 4 parts

Commit message: Signal and Cuk imported
Parts:
- added J101, J102: Conn_01x20, symbol Connector_Generic:Conn_01x20
Connections:
- wire segments 27 -> 56
- no-connect marks 0 -> 8
Changed lines of the file:
@@
 F3 "SPI_MOSI" O R 6050 5350 60
 F4 "MCP_INT" I R 6050 5550 60
-F5 "VCC" I L 4900 4950 60
-F6 "GND" O L 4900 5150 60
+F5 "VCC" I L 4900 5550 60
+F6 "GND" O L 4900 5675 60
 F7 "SPI_SCK" O R 6050 5150 50
 F8 "MCP_SS" O R 6050 5450 50
+F9 "V_Vpanel_ADC" O L 4900 4950 50
+F10 "V_Ipanel_ADC" O L 4900 4750 50
+F11 "V_Vbat_ADC" O L 4900 5050 50
+F12 "V_Ibat_ADC" O L 4900 4850 50
 $EndSheet
 Wire Wire Line
@@
 L power:+5V #PWR0102
 U 1 1 5CB14A9F
-P 4725 4925
-F 0 "#PWR0102" H 4725 4775 50  0001 C CNN
-F 1 "+5V" H 4775 5125 50  0000 C CNN
-F 2 "" H 4725 4925 50  0001 C CNN
-F 3 "" H 4725 4925 50  0001 C CNN
-	1    4725 4925
+P 4725 5525
+F 0 "#PWR0102" H 4725 5375 50  0001 C CNN
+F 1 "+5V" H 4775 5725 50  0000 C CNN
+F 2 "" H 4725 5525 50  0001 C CNN
+F 3 "" H 4725 5525 50  0001 C CNN
+	1    4725 5525
 	1    0    0    -1
 $EndComp
@@
 L power:GND #PWR0106
 U 1 1 5CB14AC2
-P 4775 5150
-F 0 "#PWR0106" H 4775 4900 50  0001 C CNN
-F 1 "GND" H 4825 5000 50  0000 C CNN
-F 2 "" H 4775 5150 50  0001 C CNN
-F 3 "" H 4775 5150 50  0001 C CNN
-	1    4775 5150
-	1    0    0    -1
-$EndComp
-Wire Wire Line
-	4775 5150 4900 5150
-Wire Wire Line
-	4900 4950 4725 4950
-Wire Wire Line
-	4725 4950 4725 4925
+P 4775 5675
+F 0 "#PWR0106" H 4775 5425 50  0001 C CNN
+F 1 "GND" H 4825 5525 50  0000 C CNN
+F 2 "" H 4775 5675 50  0001 C CNN
+F 3 "" H 4775 5675 50  0001 C CNN
+	1    4775 5675
+	1    0    0    -1
+$EndComp
+Wire Wire Line
+	4775 5675 4900 5675
+Wire Wire Line
+	4900 5550 4725 5550
+Wire Wire Line
+	4725 5550 4725 5525
+Wire Wire Line
+	4650 4750 4900 4750
+Wire Wire Line
+	4500 4850 4900 4850
+Wire Wire Line
+	4125 5050 4900 5050
+Wire Wire Line
+	4300 4950 4900 4950
 $Sheet
-S 2875 2175 1275 1025
-U 5F260F1C
-F0 "signals" 50
-F1 "signals.sch" 50
-$EndSheet
-$Sheet
-S 5050 2150 1450 1100
+S 3600 1000 1125 2275
 U 5F261197
 F0 "Sheet5F261196" 50
 F1 "cuk.sch" 50
+F2 "12V" I R 4725 1150 50
+F3 "V_Ipanel" O L 3600 3150 50
+F4 "V_Ibat" O L 3600 3050 50
+F5 "V_Vbat" O L 3600 2300 50
+F6 "5V" I R 4725 1250 50
+F7 "GND" I R 4725 1350 50
+F8 "PWM" I R 4725 1950 50
+F9 "V_Vpanel+" O L 3600 1200 50
+F10 "V_Vpanel-" O L 3600 1300 50
 $EndSheet
+$Comp
+L Connector_Generic:Conn_01x20 J101
+U 1 1 5F5858EC
+P 2550 2100
+F 0 "J101" H 2630 2092 50  0000 L CNN
+F 1 "Conn_01x20" H 2630 2001 50  0000 L CNN
+F 2 "" H 2550 2100 50  0001 C CNN
+F 3 "~" H 2550 2100 50  0001 C CNN
+	1    2550 2100
+	1    0    0    -1
+$EndComp
+$Comp
+L Connector_Generic:Conn_01x20 J102
+U 1 1 5F5877A3
+P 2600 2100
+F 0 "J102" H 2518 3217 50  0000 C CNN
+F 1 "Conn_01x20" H 2518 3126 50  0000 C CNN
+F 2 "" H 2600 2100 50  0001 C CNN
+F 3 "~" H 2600 2100 50  0001 C CNN
+	1    2600 2100
+	-1   0    0    -1
+$EndComp
+$Comp
+L power:GND #PWR0109
+U 1 1 5F58F131
+P 2125 1400
+F 0 "#PWR0109" H 2125 1150 50  0001 C CNN
+F 1 "GND" H 2125 1250 50  0000 C CNN
+F 2 "" H 2125 1400 50  0001 C CNN
+F 3 "" H 2125 1400 50  0001 C CNN
+	1    2125 1400
+	1    0    0    -1
+$EndComp
+Wire Wire Line
+	2125 1400 2350 1400
+NoConn ~ 2350 1600
+NoConn ~ 2350 1800
+NoConn ~ 2350 1900
+NoConn ~ 2350 2000
+NoConn ~ 2350 2100
+NoConn ~ 2350 1700
+NoConn ~ 2350 2200
+$Comp
+L power:GND #PWR0110
+U 1 1 5F59A737
+P 2100 2400
+F 0 "#PWR0110" H 2100 2150 50  0001 C CNN
+F 1 "GND" H 2100 2250 50  0000 C CNN
+F 2 "" H 2100 2400 50  0001 C CNN
+F 3 "" H 2100 2400 50  0001 C CNN
+	1    2100 2400
+	1    0    0    -1
+$EndComp
+Wire Wire Line
+	2100 2400 2350 2400
+Wire Wire Line
+	2350 2500 2350 2400
+Connection ~ 2350 2400
+$Comp
+L power:GND #PWR0111
+U 1 1 5F5A8E95
+P 2200 3150
+F 0 "#PWR0111" H 2200 2900 50  0001 C CNN
+F 1 "GND" H 2200 3000 50  0000 C CNN
+F 2 "" H 2200 3150 50  0001 C CNN
+F 3 "" H 2200 3150 50  0001 C CNN
+	1    2200 3150
+	1    0    0    -1
+$EndComp
+Wire Wire Line
+	2200 3150 2200 3000
+NoConn ~ 2350 2700
+Connection ~ 2200 3000
+Wire Wire Line
+	2200 3000 2350 3000
+Wire Wire Line
+	1850 3100 2350 3100
+Wire Wire Line
+	1850 2800 2350 2800
+Wire Wire Line
+	1850 2600 2350 2600
+Wire Wire Line
+	1850 2300 2350 2300
+Wire Wire Line
+	1850 2900 2350 2900
+Wire Wire Line
+	1850 3000 2200 3000
+$Sheet
+S 1200 975  650  2475
+U 5F4FF1E4
+F0 "Signal" 50
+F1 "Signal.sch" 50
+F2 "V_Vpanel-" I R 1850 1300 50
+F3 "GND" I R 1850 3000 50
+F4 "V_Vpanel_ADC" O R 1850 1500 50
+F5 "V_Vpanel+" I R 1850 1200 50
+F6 "PWM" I R 1850 2900 50
+F7 "V_Vbat" O R 1850 2300 50
+F8 "V_Vbat_ADC" O R 1850 2600 50
+F9 "BatOVInterrupt" O R 1850 2800 50
+F10 "+5V" I R 1850 3100 50
+$EndSheet
+Wire Wire Line
+	1850 1500 2350 1500
+Wire Wire Line
+	1850 1300 2350 1300
+Wire Wire Line
+	1850 1200 2350 1200
+Wire Wire Line
+	2800 1200 3600 1200
+Wire Wire Line
+	3600 1300 2800 1300
+Wire Wire Line
+	3600 2300 2800 2300
+Wire Wire Line
+	2800 1500 3150 1500
+Wire Wire Line
+	2800 2600 2975 2600
+Wire Wire Line
+	3150 1500 3150 4425
+Wire Wire Line
+	2975 2600 2975 4525
+Wire Wire Line
+	3600 3150 3500 3150
+Wire Wire Line
+	3500 3150 3500 4225
+Wire Wire Line
+	3600 3050 3350 3050
+Wire Wire Line
+	3350 3050 3350 4325
 $EndSCHEMATC

Commit message: schematic and footprint
Parts:
- added U101, U102: ZCS, KicadZeniteSolarLibrary18:ZCS18, symbol ZCS:ZCS
- J101: footprint (none) -> Connector_PinHeader_2.54mm:PinHeader_1x20_P2.54mm_Horizontal
- J102: footprint (none) -> Connector_PinSocket_2.54mm:PinSocket_1x20_P2.54mm_Vertical
Connections:
- net labels added: +12V, +5P, BatOVInterrupt, GNDPWR, GNDS, PWM, VCC, VCCQ
- wire segments 56 -> 136
- no-connect marks 8 -> 16
Other:
- note added: "SIGNALS\n"
- note added: "ZCS"
