File: hardware/MCC20.sch (KiCad schematic (older format))
At the start: 8 parts, among them J101 Conn_01x20, J102 Conn_01x20, U101 ZCS, U102 ZCS

Commit message: parte de potencia
Connections:
- net GNDPWR: now also U101.18 (GND), U101.2 (GND), U101.22 (GND), U101.25 (GND), U101.28 (GND), U101.3 (GND), U101.37 (GNDA), U101.4 (GND), U101.6 (GND), U101.7 (GND), U101.8 (GND)
Changed lines of the file:
@@
 Wire Wire Line
 	2800 2600 3075 2600
+$Comp
+L power:GNDPWR #PWR0151
+U 1 1 5F5527DF
+P 4375 4350
+F 0 "#PWR0151" H 4375 4150 50  0001 C CNN
+F 1 "GNDPWR" H 4379 4196 50  0000 C CNN
+F 2 "" H 4375 4300 50  0001 C CNN
+F 3 "" H 4375 4300 50  0001 C CNN
+	1    4375 4350
+	1    0    0    -1
+$EndComp
+Wire Wire Line
+	4375 4350 4375 4325
+Wire Wire Line
+	4375 4325 4450 4325
 $EndSCHEMATC

Commit message: snubber
Parts:
- J102: footprint Connector_PinSocket_2.54mm:PinSocket_1x20_P2.54mm_Vertical -> Connector_PinSocket_2.54mm:PinSocket_1x20_P2.54mm_Vertical_SMD_Pin1Left
Changed lines of the file:
@@
 F 0 "J102" H 2518 3217 50  0000 C CNN
 F 1 "Conn_01x20" H 2518 3126 50  0000 C CNN
-F 2 "Connector_PinSocket_2.54mm:PinSocket_1x20_P2.54mm_Vertical" H 2600 2100 50  0001 C CNN
+F 2 "Connector_PinSocket_2.54mm:PinSocket_1x20_P2.54mm_Vertical_SMD_Pin1Left" H 2600 2100 50  0001 C CNN
 F 3 "~" H 2600 2100 50  0001 C CNN
 	1    2600 2100
