File: hardware/Signal.sch (KiCad schematic (older format))
At the start: 23 parts, among them Q702 Q_NPN_Darlington_BEC, U703 LM324, U704 INA826

Commit message: schematic and footprint
Parts:
- U704: footprint (none) -> Package_SO:SOIC-8_3.9x4.9mm_P1.27mm
Changed lines of the file:
@@
 $Descr A4 11693 8268
 encoding utf-8
-Sheet 7 7
+Sheet 6 8
 Title ""
 Date ""
@@
 F 0 "U704" H 5275 4975 50  0000 L CNN
 F 1 "INA826" H 5250 4900 50  0000 L CNN
-F 2 "" H 5275 4775 50  0001 C CNN
+F 2 "Package_SO:SOIC-8_3.9x4.9mm_P1.27mm" H 5275 4775 50  0001 C CNN
 F 3 "http://www.ti.com/lit/ds/symlink/ina826.pdf" H 5275 4775 50  0001 C CNN
 	1    5175 4775
