File: hardware/atmega328p.sch (KiCad schematic (older format))
At the start: 17 parts, among them J401 USART, U401 ATMEGA328P-PU, Y401 16MHz

Commit message: Signal and Cuk imported
Connections:
- net V_Vpanel_ADC: now reaches U401.23 (PC0)
- net V_Ipanel_ADC: now reaches U401.24 (PC1)
- net V_Vbat_ADC: now reaches U401.25 (PC2)
- net V_Ibat_ADC: now reaches U401.26 (PC3)
- net SCL: no longer names the net of U401.28 (PC5)
- net SDA: no longer names the net of U401.27 (PC4)
- no-connect marks 9 -> 7
Changed lines of the file:
@@
 $Descr A4 11693 8268
 encoding utf-8
-Sheet 3 7
+Sheet 5 7
 Title ""
 Date ""
@@
 AR Path="/5F24EEA3/5F253E29/59FE3A5A" Ref="Y?"  Part="1"
 AR Path="/5F24EEA3/5F256CB5/59FE3A5A" Ref="Y?"  Part="1"
-F 0 "Y?" H 8300 3700 50  0000 C CNN
+F 0 "Y401" H 8300 3700 50  0000 C CNN
 F 1 "16MHz" H 8300 3500 50  0000 C CNN
 F 2 "Crystal:Crystal_HC49-U_Vertical" H 8300 3600 50  0001 C CNN
@@
 AR Path="/5F24EEA3/5F253E29/59FE3A61" Ref="C?"  Part="1"
 AR Path="/5F24EEA3/5F256CB5/59FE3A61" Ref="C?"  Part="1"
-F 0 "C?" H 8060 3870 50  0000 L CNN
+F 0 "C403" H 8060 3870 50  0000 L CNN
 F 1 "22pF" H 8060 3720 50  0000 L CNN
 F 2 "Capacitor_SMD:C_0805_2012Metric_Pad1.15x1.40mm_HandSolder" H 8050 3800 50  0001 C CNN
@@
 AR Path="/5F24EEA3/5F253E29/59FE3A68" Ref="C?"  Part="1"
 AR Path="/5F24EEA3/5F256CB5/59FE3A68" Ref="C?"  Part="1"
-F 0 "C?" H 8350 3900 50  0000 L CNN
+F 0 "C404" H 8350 3900 50  0000 L CNN
 F 1 "22pF" H 8350 3700 50  0000 L CNN
 F 2 "Capacitor_SMD:C_0805_2012Metric_Pad1.15x1.40mm_HandSolder" H 8550 3800 50  0001 C CNN
@@
 AR Path="/5F24EEA3/5F253E29/59FE4B17" Ref="R?"  Part="1"
 AR Path="/5F24EEA3/5F256CB5/59FE4B17" Ref="R?"  Part="1"
-F 0 "R?" H 6030 4070 50  0000 L CNN
+F 0 "R401" H 6030 4070 50  0000 L CNN
 F 1 "10k" H 6030 4010 50  0000 L CNN
 F 2 "Resistor_SMD:R_0805_2012Metric_Pad1.15x1.40mm_HandSolder" H 6000 4050 50  0001 C CNN
@@
 AR Path="/5F24EEA3/5F253E29/59FE4EE2" Ref="C?"  Part="1"
 AR Path="/5F24EEA3/5F256CB5/59FE4EE2" Ref="C?"  Part="1"
-F 0 "C?" V 5900 4350 50  0000 L CNN
+F 0 "C406" V 5900 4350 50  0000 L CNN
 F 1 "100nF" V 6050 4500 50  0000 L CNN
 F 2 "Capacitor_SMD:C_0805_2012Metric_Pad1.15x1.40mm_HandSolder" H 6000 4450 50  0001 C CNN
@@
 AR Path="/5F24EEA3/5F253E29/59FE5354" Ref="D?"  Part="1"
 AR Path="/5F24EEA3/5F256CB5/59FE5354" Ref="D?"  Part="1"
-F 0 "D?" H 5850 5625 50  0000 L CNN
+F 0 "D402" H 5850 5625 50  0000 L CNN
 F 1 "LED_RED" H 5800 5400 50  0000 L CNN
 F 2 "LED_SMD:LED_0805_2012Metric_Pad1.15x1.40mm_HandSolder" V 5900 5500 50  0001 C CNN
@@
 AR Path="/5F24EEA3/5F253E29/59FFC489" Ref="R?"  Part="1"
 AR Path="/5F24EEA3/5F256CB5/59FFC489" Ref="R?"  Part="1"
-F 0 "R?" H 5930 5220 50  0000 L CNN
+F 0 "R404" H 5930 5220 50  0000 L CNN
 F 1 "1k" H 5930 5160 50  0000 L CNN
 F 2 "Resistor_SMD:R_0805_2012Metric_Pad1.15x1.40mm_HandSolder" H 5900 5200 50  0001 C CNN
@@
 AR Path="/5F24EEA3/5F253E29/5AACAE36" Ref="R?"  Part="1"
 AR Path="/5F24EEA3/5F256CB5/5AACAE36" Ref="R?"  Part="1"
-F 0 "R?" V 7400 4450 50  0000 L CNN
+F 0 "R402" V 7400 4450 50  0000 L CNN
 F 1 "1k" V 7400 4200 50  0000 L CNN
 F 2 "Resistor_SMD:R_0805_2012Metric_Pad1.15x1.40mm_HandSolder" H 7350 4350 50  0001 C CNN
@@
 AR Path="/5F24EEA3/5F253E29/5AACB0BA" Ref="R?"  Part="1"
 AR Path="/5F24EEA3/5F256CB5/5AACB0BA" Ref="R?"  Part="1"
-F 0 "R?" V 7400 4550 50  0000 L CNN
+F 0 "R403" V 7400 4550 50  0000 L CNN
 F 1 "1k" V 7400 4300 50  0000 L CNN
 F 2 "Resistor_SMD:R_0805_2012Metric_Pad1.15x1.40mm_HandSolder" H 7350 4450 50  0001 C CNN
@@
 	0    -1   -1   0
 $EndComp
-Text HLabel 5050 4150 2    60   Input ~ 0
-SCL
-NoConn ~ 5050 3850
-NoConn ~ 5050 3950
 NoConn ~ 5050 4750
 NoConn ~ 5050 4650
@@
 Wire Wire Line
 	5900 5300 5900 5400
-NoConn ~ 5050 3750
 Wire Wire Line
 	4350 5450 4350 5650
@@
 AR Path="/5F24EEA3/5F253E29/5BE7DD75" Ref="D?"  Part="1"
 AR Path="/5F24EEA3/5F256CB5/5BE7DD75" Ref="D?"  Part="1"
-F 0 "D?" H 6150 5625 50  0000 L CNN
+F 0 "D403" H 6150 5625 50  0000 L CNN
 F 1 "LED_RED" H 6100 5400 50  0000 L CNN
 F 2 "LED_SMD:LED_0805_2012Metric_Pad1.15x1.40mm_HandSolder" V 6200 5500 50  0001 C CNN
@@
 AR Path="/5F24EEA3/5F253E29/5BE7DD7B" Ref="R?"  Part="1"
 AR Path="/5F24EEA3/5F256CB5/5BE7DD7B" Ref="R?"  Part="1"
-F 0 "R?" H 6230 5220 50  0000 L CNN
+F 0 "R405" H 6230 5220 50  0000 L CNN
 F 1 "1k" H 6230 5160 50  0000 L CNN
 F 2 "Resistor_SMD:R_0805_2012Metric_Pad1.15x1.40mm_HandSolder" H 6200 5200 50  0001 C CNN
@@
 AR Path="/5F24EEA3/5F253E29/5BE95CC8" Ref="D?"  Part="1"
 AR Path="/5F24EEA3/5F256CB5/5BE95CC8" Ref="D?"  Part="1"
-F 0 "D?" V 5650 4200 50  0000 R CNN
+F 0 "D401" V 5650 4200 50  0000 R CNN
 F 1 "LL4148" V 6025 4200 50  0000 R CNN
 F 2 "Diode_SMD:D_MiniMELF_Handsoldering" H 5750 3875 50  0001 C CNN
@@
 AR Path="/5F24EEA3/5F253E29/5BEB6AE8" Ref="#PWR0107"  Part="1"
 AR Path="/5F24EEA3/5F256CB5/5BEB6AE8" Ref="#PWR?"  Part="1"
-F 0 "#PWR?" H 8300 3850 50  0001 C CNN
+F 0 "#PWR0407" H 8300 3850 50  0001 C CNN
 F 1 "GND" H 8350 3900 50  0000 C CNN
 F 2 "" H 8300 4100 50  0001 C CNN
@@
 AR Path="/5F24EEA3/5F253E29/5BEB7AB4" Ref="#PWR0108"  Part="1"
 AR Path="/5F24EEA3/5F256CB5/5BEB7AB4" Ref="#PWR?"  Part="1"
-F 0 "#PWR?" H 4350 5500 50  0001 C CNN
+F 0 "#PWR0412" H 4350 5500 50  0001 C CNN
 F 1 "GND" H 4400 5550 50  0000 C CNN
 F 2 "" H 4350 5750 50  0001 C CNN
@@
 AR Path="/5F24EEA3/5F253E29/5BEC895B" Ref="#PWR0109"  Part="1"
 AR Path="/5F24EEA3/5F256CB5/5BEC895B" Ref="#PWR?"  Part="1"
-F 0 "#PWR?" H 8050 2200 50  0001 C CNN
+F 0 "#PWR0404" H 8050 2200 50  0001 C CNN
 F 1 "GND" H 8100 2250 50  0000 C CNN
 F 2 "" H 8050 2450 50  0001 C CNN
@@
 AR Path="/5F24EEA3/5F253E29/5BECD3FE" Ref="J?"  Part="1"
 AR Path="/5F24EEA3/5F256CB5/5BECD3FE" Ref="J?"  Part="1"
-F 0 "J?" H 7700 4000 50  0000 C CNN
+F 0 "J401" H 7700 4000 50  0000 C CNN
 F 1 "USART" H 7700 4100 50  0000 C CNN
 F 2 "Connector_PinHeader_2.54mm:PinHeader_1x04_P2.54mm_Vertical" H 7750 4450 50  0001 C CNN
@@
 AR Path="/5F24EEA3/5F253E29/5BECF494" Ref="#PWR0110"  Part="1"
 AR Path="/5F24EEA3/5F256CB5/5BECF494" Ref="#PWR?"  Part="1"
-F 0 "#PWR?" H 6000 4400 50  0001 C CNN
+F 0 "#PWR0408" H 6000 4400 50  0001 C CNN
 F 1 "GND" H 6050 4450 50  0000 C CNN
 F 2 "" H 6000 4650 50  0001 C CNN
@@
 AR Path="/5F24EEA3/5F253E29/5BED8033" Ref="C?"  Part="1"
 AR Path="/5F24EEA3/5F256CB5/5BED8033" Ref="C?"  Part="1"
-F 0 "C?" V 6200 4100 50  0000 L CNN
+F 0 "C405" V 6200 4100 50  0000 L CNN
 F 1 "100nF" V 6100 4000 50  0000 L CNN
 F 2 "Capacitor_SMD:C_0805_2012Metric_Pad1.15x1.40mm_HandSolder" H 6300 4250 50  0001 C CNN
@@
 AR Path="/5F24EEA3/5F253E29/5BEE0905" Ref="#PWR0111"  Part="1"
 AR Path="/5F24EEA3/5F256CB5/5BEE0905" Ref="#PWR?"  Part="1"
-F 0 "#PWR?" H 7450 4400 50  0001 C CNN
+F 0 "#PWR0409" H 7450 4400 50  0001 C CNN
 F 1 "GND" H 7500 4450 50  0000 C CNN
 F 2 "" H 7450 4650 50  0001 C CNN
@@
 AR Path="/5F24EEA3/5F253E29/5BF321D4" Ref="#PWR0112"  Part="1"
 AR Path="/5F24EEA3/5F256CB5/5BF321D4" Ref="#PWR?"  Part="1"
-F 0 "#PWR?" H 4350 1600 50  0001 C CNN
+F 0 "#PWR0401" H 4350 1600 50  0001 C CNN
 F 1 "+5V" H 4400 1950 50  0000 C CNN
 F 2 "" H 4350 1750 50  0001 C CNN
@@
 AR Path="/5F24EEA3/5F253E29/5BF32222" Ref="#PWR0113"  Part="1"
 AR Path="/5F24EEA3/5F256CB5/5BF32222" Ref="#PWR?"  Part="1"
-F 0 "#PWR?" H 8050 2000 50  0001 C CNN
+F 0 "#PWR0402" H 8050 2000 50  0001 C CNN
 F 1 "+5V" H 8100 2350 50  0000 C CNN
 F 2 "" H 8050 2150 50  0001 C CNN
@@
 AR Path="/5F24EEA3/5F253E29/5BF330B7" Ref="#PWR0114"  Part="1"
 AR Path="/5F24EEA3/5F256CB5/5BF330B7" Ref="#PWR?"  Part="1"
-F 0 "#PWR?" H 5750 3600 50  0001 C CNN
+F 0 "#PWR0406" H 5750 3600 50  0001 C CNN
 F 1 "+5V" H 5800 3950 50  0000 C CNN
 F 2 "" H 5750 3750 50  0001 C CNN
@@
 AR Path="/5F24EEA3/5F253E29/5BF3B4C1" Ref="C?"  Part="1"
 AR Path="/5F24EEA3/5F256CB5/5BF3B4C1" Ref="C?"  Part="1"
-F 0 "C?" H 3700 2850 50  0000 L CNN
+F 0 "C402" H 3700 2850 50  0000 L CNN
 F 1 "100nF" H 3700 3050 50  0000 L CNN
 F 2 "Capacitor_SMD:C_0805_2012Metric_Pad1.15x1.40mm_HandSolder" H 3650 2950 50  0001 C CNN
@@
 AR Path="/5F24EEA3/5F253E29/5BF3D2B5" Ref="#PWR0115"  Part="1"
 AR Path="/5F24EEA3/5F256CB5/5BF3D2B5" Ref="#PWR?"  Part="1"
-F 0 "#PWR?" H 3650 2900 50  0001 C CNN
+F 0 "#PWR0405" H 3650 2900 50  0001 C CNN
 F 1 "GND" H 3700 2950 50  0000 C CNN
 F 2 "" H 3650 3150 50  0001 C CNN
@@
 AR Path="/5F24EEA3/5F253E29/5BF2780D" Ref="C?"  Part="1"
 AR Path="/5F24EEA3/5F256CB5/5BF2780D" Ref="C?"  Part="1"
-F 0 "C?" H 4650 2050 50  0000 L CNN
+F 0 "C401" H 4650 2050 50  0000 L CNN
 F 1 "100nF" H 4550 2150 50  0000 L CNN
 F 2 "Capacitor_SMD:C_0805_2012Metric_Pad1.15x1.40mm_HandSolder" H 4550 2050 50  0001 C CNN
@@
 AR Path="/5F24EEA3/5F253E29/5BF3B38D" Ref="#PWR0116"  Part="1"
 AR Path="/5F24EEA3/5F256CB5/5BF3B38D" Ref="#PWR?"  Part="1"
-F 0 "#PWR?" H 4550 2000 50  0001 C CNN
+F 0 "#PWR0403" H 4550 2000 50  0001 C CNN
 F 1 "GND" H 4600 2050 50  0000 C CNN
 F 2 "" H 4550 2250 50  0001 C CNN
@@
 AR Path="/5F24EEA3/5F253E29/59FE3414" Ref="U?"  Part="1"
 AR Path="/5F24EEA3/5F256CB5/59FE3414" Ref="U?"  Part="1"
-F 0 "U?" H 3850 5400 50  0000 L BNN
+F 0 "U401" H 3850 5400 50  0000 L BNN
 F 1 "ATMEGA328P-PU" H 4500 2450 50  0000 L BNN
 F 2 "Package_DIP:DIP-28_W7.62mm_Socket" H 4350 3950 50  0001 C CIN
@@
 	1    0    0    -1
 $EndComp
-Text HLabel 5050 4050 2    60   Input ~ 0
-SDA
-NoConn ~ 5050 3650
+NoConn ~ 5050 4050
+NoConn ~ 5050 4150
+Text HLabel 5050 3650 2    50   Output ~ 0
+V_Vpanel_ADC
+Text HLabel 5050 3750 2    50   Output ~ 0
+V_Ipanel_ADC
+Text HLabel 5050 3850 2    50   Output ~ 0
+V_Vbat_ADC
+Text HLabel 5050 3950 2    50   Output ~ 0
+V_Ibat_ADC
 $EndSCHEMATC

Commit message: schematic and footprint
Connections:
- net PWM: now reaches U401.16 (PB2)
- no-connect marks 7 -> 6
Changed lines of the file:
@@
 $Descr A4 11693 8268
 encoding utf-8
-Sheet 5 7
+Sheet 4 8
 Title ""
 Date ""
@@
 Wire Wire Line
 	5050 2950 4950 2950
-NoConn ~ 5050 2950
 Text Label 5300 2850 0    60   ~ 0
 MCP_INT
@@
 Text HLabel 5050 3950 2    50   Output ~ 0
 V_Ibat_ADC
+Text HLabel 5050 2950 2    50   Output ~ 0
+PWM
 $EndSCHEMATC
