File: hardware/cuk.sch (KiCad schematic (older format))
At the start: 73 parts

Commit message: Signal and Cuk imported
Parts:
- removed JP? (x2): Diode On, Jumper:SolderJumper-2_P1.3mm_Open_Pad1.0x1.5mm, symbol Device:Jumper_NC_Small
- removed JP?: MosfetOn, Jumper:SolderJumper-2_P1.3mm_Open_TrianglePad1.0x1.5mm, symbol Device:Jumper_NC_Small
- removed R?: G=1+(49.4k/Rg), symbol Device:R_US
- removed R? (x3): ?, symbol Device:R_US
- removed Rg?: 10k, Resistor_SMD:R_0805_2012Metric_Pad1.15x1.40mm_HandSolder, symbol Device:R_Small
- removed U?: INA826, symbol KicadZeniteSolarLibrary:INA826
- added R703: 560k, symbol Device:R_US
- added R704: 39k, symbol Device:R_US
- R701, R702: renamed from R?; value ? -> 330k
- gave numbers to parts that had none: 62
Connections:
- net labels added: 5V, V_Vbat, V_Vpanel+, V_Vpanel-
- net labels removed: +5VA, LG, V_Vpanel
- wire segments 222 -> 204
- no-connect marks 0 -> 2
Other:
- moved on the sheet: C701, C702, R701, R702, Tvs701, Tvs702, U701, U702

Commit message: schematic and footprint
Parts:
- D701: footprint MCCplaca:TO-247-3_Horizontal_TabUp -> KicadZeniteSolarLibrary18:TO-247-3_Horizontal_TabUp
- F701: footprint MCCplaca:Porta_Fusivel -> KicadZeniteSolarLibrary18:Porta_Fusivel
- HS701: footprint MCCplaca:hs10425 -> KicadZeniteSolarLibrary18:hs10425
- J701: footprint (none) -> KicadZeniteSolarLibrary18:Driver_(INEP)
- L1/701, L2/701: footprint MCCplaca:Inductor_Nocoupled -> KicadZeniteSolarLibrary18:Inductor_Nocoupled
- R701, R702, R703, R704: footprint (none) -> Resistor_SMD:R_0805_2012Metric_Pad1.15x1.40mm_HandSolder
- Rshunt701, Rshunt702: footprint MCCplaca Shunt:PML100HZPJV0L5 -> Resistor_SMD:R_2512_6332Metric_Pad1.52x3.35mm_HandSolder
Changed lines of the file:
@@
 $Descr A4 11693 8268
 encoding utf-8
-Sheet 6 7
+Sheet 5 8
 Title ""
 Date ""
@@
 F 0 "HS701" H 4892 1171 50  0000 L CNN
 F 1 "Heatsink" H 4892 1080 50  0000 L CNN
-F 2 "MCCplaca:hs10425" H 4762 1050 50  0001 C CNN
+F 2 "KicadZeniteSolarLibrary18:hs10425" H 4762 1050 50  0001 C CNN
 F 3 "" H 4762 1050 50  0001 C CNN
 	1    4750 1050
@@
 F 0 "F701" H 8060 4396 50  0000 L CNN
 F 1 "Fuse" H 8060 4305 50  0000 L CNN
-F 2 "MCCplaca:Porta_Fusivel" V 7930 4350 50  0001 C CNN
+F 2 "KicadZeniteSolarLibrary18:Porta_Fusivel" V 7930 4350 50  0001 C CNN
 F 3 "" H 8000 4350 50  0001 C CNN
 	1    8000 4350
@@
 F 0 "D701" V 3950 2700 50  0000 L CNN
 F 1 "80CPQ150PbF" V 4100 2700 50  0000 L CNN
-F 2 "MCCplaca:TO-247-3_Horizontal_TabUp" H 4100 2650 50  0001 C CNN
+F 2 "KicadZeniteSolarLibrary18:TO-247-3_Horizontal_TabUp" H 4100 2650 50  0001 C CNN
 F 3 "https://www.vishay.com/docs/94257/vs-80cpq150.pdf" H 4100 2650 50  0001 C CNN
 	1    4100 2650
@@
 F 0 "Rshunt702" H 8070 3946 50  0000 L CNN
 F 1 "1500uR" H 8070 3855 50  0000 L CNN
-F 2 "MCCplaca Shunt:PML100HZPJV0L5" V 7930 3900 50  0001 C CNN
+F 2 "Resistor_SMD:R_2512_6332Metric_Pad1.52x3.35mm_HandSolder" V 7930 3900 50  0001 C CNN
 F 3 "~" H 8000 3900 50  0001 C CNN
 	1    8000 3900
@@
 F 0 "L1/701" H 5150 1650 50  0000 L CNN
 F 1 "L_Core_Iron_Small" H 5118 1605 50  0001 L CNN
-F 2 "MCCplaca:Inductor_Nocoupled" H 5050 1650 50  0001 C CNN
+F 2 "KicadZeniteSolarLibrary18:Inductor_Nocoupled" H 5050 1650 50  0001 C CNN
 F 3 "~" H 5050 1650 50  0001 C CNN
 	1    5050 1650
@@
 F 0 "L2/701" H 5600 1650 50  0000 R CNN
 F 1 "L_Core_Iron_Small" H 5309 1695 50  0001 R CNN
-F 2 "MCCplaca:Inductor_Nocoupled" H 5350 1650 50  0001 C CNN
+F 2 "KicadZeniteSolarLibrary18:Inductor_Nocoupled" H 5350 1650 50  0001 C CNN
 F 3 "~" H 5350 1650 50  0001 C CNN
 	1    5350 1650
@@
 F 0 "J701" H 10680 3667 50  0000 L CNN
 F 1 "Driver_INEP" H 10680 3576 50  0000 L CNN
-F 2 "" H 10600 3625 50  0001 C CNN
+F 2 "KicadZeniteSolarLibrary18:Driver_(INEP)" H 10600 3625 50  0001 C CNN
 F 3 "~" H 10600 3625 50  0001 C CNN
 	1    10600 3625
@@
 F 0 "Rshunt701" H 4120 3996 50  0000 L CNN
 F 1 "1500uR" H 4120 3905 50  0000 L CNN
-F 2 "MCCplaca Shunt:PML100HZPJV0L5" V 3980 3950 50  0001 C CNN
+F 2 "Resistor_SMD:R_2512_6332Metric_Pad1.52x3.35mm_HandSolder" V 3980 3950 50  0001 C CNN
 F 3 "~" H 4050 3950 50  0001 C CNN
 	1    4050 3950
@@
 F 0 "R703" H 10518 5871 50  0000 L CNN
 F 1 "560k" H 10525 5950 50  0000 L CNN
-F 2 "" V 10490 5815 50  0001 C CNN
+F 2 "Resistor_SMD:R_0805_2012Metric_Pad1.15x1.40mm_HandSolder" V 10490 5815 50  0001 C CNN
 F 3 "~" H 10450 5825 50  0001 C CNN
 	1    10450 5825
@@
 F 0 "R704" H 10693 6021 50  0000 L CNN
 F 1 "39k" H 10700 6100 50  0000 L CNN
-F 2 "" V 10665 5965 50  0001 C CNN
+F 2 "Resistor_SMD:R_0805_2012Metric_Pad1.15x1.40mm_HandSolder" V 10665 5965 50  0001 C CNN
 F 3 "~" H 10625 5975 50  0001 C CNN
 	1    10625 5975
@@
 F 0 "R701" H 9275 6225 50  0000 L CNN
 F 1 "330k" H 9250 6150 50  0000 L CNN
-F 2 "" V 9240 6215 50  0001 C CNN
+F 2 "Resistor_SMD:R_0805_2012Metric_Pad1.15x1.40mm_HandSolder" V 9240 6215 50  0001 C CNN
 F 3 "~" H 9200 6225 50  0001 C CNN
 	1    9200 6225
@@
 F 0 "R702" H 9293 5896 50  0000 L CNN
 F 1 "330k" H 9300 5975 50  0000 L CNN
-F 2 "" V 9265 5840 50  0001 C CNN
+F 2 "Resistor_SMD:R_0805_2012Metric_Pad1.15x1.40mm_HandSolder" V 9265 5840 50  0001 C CNN
 F 3 "~" H 9225 5850 50  0001 C CNN
 	1    9225 5850
