File: hardware/cuk.sch (KiCad schematic (older format))
At the start: 66 parts, among them J701 Driver_INEP, Q701 IRFP4321PbF, U701 INA240A4D, U702 INA240A4D

Commit message: snubber
Parts:
- J701: footprint KicadZeniteSolarLibrary18:Driver_(INEP) -> KicadZeniteSolarLibrary18:Driver_(INEP)_SMD
- Rshunt701, Rshunt702: footprint Resistor_SMD:R_2512_6332Metric_Pad1.52x3.35mm_HandSolder -> KicadZeniteSolarLibrary18:PML100HZPJV0L5
Connections:
- net +B: now also L1/701.2; no longer L1/701.1
- net -Vp: now also L2/701.1; no longer L2/701.2
- net HS: now also L1/701.1, L2/701.2; no longer L1/701.2, L2/701.1
Changed lines of the file:
@@
 F 0 "Rshunt702" H 8070 3946 50  0000 L CNN
 F 1 "1500uR" H 8070 3855 50  0000 L CNN
-F 2 "Resistor_SMD:R_2512_6332Metric_Pad1.52x3.35mm_HandSolder" V 7930 3900 50  0001 C CNN
+F 2 "KicadZeniteSolarLibrary18:PML100HZPJV0L5" V 7930 3900 50  0001 C CNN
 F 3 "~" H 8000 3900 50  0001 C CNN
 	1    8000 3900
@@
 F 3 "~" H 5050 1650 50  0001 C CNN
 	1    5050 1650
-	-1   0    0    -1
+	-1   0    0    1
 $EndComp
 $Comp
@@
 F 3 "~" H 5350 1650 50  0001 C CNN
 	1    5350 1650
-	1    0    0    1
+	1    0    0    -1
 $EndComp
 Wire Wire Line
@@
 F 0 "J701" H 10680 3667 50  0000 L CNN
 F 1 "Driver_INEP" H 10680 3576 50  0000 L CNN
-F 2 "KicadZeniteSolarLibrary18:Driver_(INEP)" H 10600 3625 50  0001 C CNN
+F 2 "KicadZeniteSolarLibrary18:Driver_(INEP)_SMD" H 10600 3625 50  0001 C CNN
 F 3 "~" H 10600 3625 50  0001 C CNN
 	1    10600 3625
@@
 F 0 "Rshunt701" H 4120 3996 50  0000 L CNN
 F 1 "1500uR" H 4120 3905 50  0000 L CNN
-F 2 "Resistor_SMD:R_2512_6332Metric_Pad1.52x3.35mm_HandSolder" V 3980 3950 50  0001 C CNN
+F 2 "KicadZeniteSolarLibrary18:PML100HZPJV0L5" V 3980 3950 50  0001 C CNN
 F 3 "~" H 4050 3950 50  0001 C CNN
 	1    4050 3950
