File: hardware/_autosave-cuk.sch (KiCad schematic (older format))
At the start: 66 parts, among them J701 Driver_INEP, Q701 IRFP4321PbF, U701 INA240A4D, U702 INA240A4D

Commit message: parte de potencia
Parts:
- Rshunt701, Rshunt702: footprint Resistor_SMD:R_2512_6332Metric_Pad1.52x3.35mm_HandSolder -> KicadZeniteSolarLibrary18:PML100HZPJV0L5
Changed lines of the file:
@@
 F 0 "Rshunt702" H 8070 3946 50  0000 L CNN
 F 1 "1500uR" H 8070 3855 50  0000 L CNN
-F 2 "Resistor_SMD:R_2512_6332Metric_Pad1.52x3.35mm_HandSolder" V 7930 3900 50  0001 C CNN
+F 2 "KicadZeniteSolarLibrary18:PML100HZPJV0L5" V 7930 3900 50  0001 C CNN
 F 3 "~" H 8000 3900 50  0001 C CNN
 	1    8000 3900
@@
 F 0 "Rshunt701" H 4120 3996 50  0000 L CNN
 F 1 "1500uR" H 4120 3905 50  0000 L CNN
-F 2 "Resistor_SMD:R_2512_6332Metric_Pad1.52x3.35mm_HandSolder" V 3980 3950 50  0001 C CNN
+F 2 "KicadZeniteSolarLibrary18:PML100HZPJV0L5" V 3980 3950 50  0001 C CNN
 F 3 "~" H 4050 3950 50  0001 C CNN
 	1    4050 3950
