File: hardware/MCC20.kicad_pcb (KiCad board)
At the start: 2 copper layers, 247.1 x 121 mm, 212 parts, among them J1 Conn_01x04, J401 USART, J601 RJ45, J602 RJ45, U201 MCP2551-I/SN, U202 MCP2515-xSO, U401 ATMEGA328P-PU, U501 LM7805, Y201 16MHz, Y401 16MHz

Commit message: Signal and Cuk imported
Parts:
- removed the C102 at (237.5, 43.4)
- removed the C102 at (172.5, 43.4)
- removed the C102 at (107.5, 43.4)
- removed the C201 at (235.0, 94.0)
- removed the C201 at (170.0, 94.0)
- removed the C201 at (105.0, 94.0)
- removed the C202 at (242.6, 109.9)
- removed the C202 at (177.6, 109.9)
- removed the C202 at (112.6, 109.9)
- removed the C203 at (227.4, 100.1)
- removed the C203 at (162.4, 100.1)
- removed the C203 at (97.4, 100.1)
- removed the C204 at (229.5, 96.3)
- removed the C204 at (164.5, 96.3)
- removed the C204 at (99.5, 96.3)
- removed the C205 at (237.8, 119.8)
- removed the C205 at (172.8, 119.8)
- removed the C205 at (107.8, 119.8)
- removed the C401 at (246.1, 73.4)
- removed the C401 at (181.1, 73.4)
- removed the C401 at (116.1, 73.4)
- removed the C402 at (230.8, 68.3)
- removed the C402 at (165.8, 68.3)
- removed the C402 at (100.8, 68.3)
- removed the C403 at (228.3, 75.9)
- removed the C403 at (163.3, 75.9)
- removed the C403 at (98.3, 75.9)
- removed the C404 at (229.5, 71.5)
- removed the C404 at (164.5, 71.5)
- removed the C404 at (99.5, 71.5)
- removed the C405 at (229.5, 53.1)
- removed the C405 at (164.5, 53.1)
- removed the C405 at (99.5, 53.1)
- removed the C406 at (232.0, 48.1)
- removed the C406 at (167.0, 48.1)
- removed the C406 at (102.0, 48.1)
- removed the C501 at (258.1, 95.9)
- removed the C501 at (193.1, 95.9)
- removed the C501 at (128.1, 95.9)
- removed the C502 at (258.1, 92.1)
- removed the C502 at (193.1, 92.1)
- removed the C502 at (128.1, 92.1)
- removed the C503 at (251.5, 95.2)
- removed the C503 at (186.5, 95.2)
- removed the C503 at (121.5, 95.2)
- removed the C504 at (251.5, 92.1)
- removed the C504 at (186.5, 92.1)
- removed the C504 at (121.5, 92.1)
- removed the D201 at (246.1, 124.8)
- removed the D201 at (181.1, 124.8)
- removed the D201 at (116.1, 124.8)
- removed the D401 at (225.0, 48.3)
- removed the D401 at (160.0, 48.3)
- removed the D401 at (95.0, 48.3)
- removed the D402 at (224.5, 88.4)
- removed the D402 at (159.5, 88.4)
- removed the D402 at (94.5, 88.4)
- removed the D403 at (224.5, 85.8)
- removed the D403 at (159.5, 85.8)
- removed the D403 at (94.5, 85.8)
- removed the D501 at (263.6, 109.2)
- removed the D501 at (198.6, 109.2)
- removed the D501 at (133.6, 109.2)
- removed the F501 at (263.6, 100.3)
- removed the F501 at (198.6, 100.3)
- removed the F501 at (133.6, 100.3)
- removed the H101 at (222.9, 38.1)
- removed the H101 at (157.9, 38.1)
- removed the H101 at (92.9, 38.1)
- removed the H102 at (221.9, 122.9)
- removed the H102 at (156.9, 122.9)
- removed the H102 at (91.9, 122.9)
- removed the H103 at (265.1, 122.9)
- removed the H103 at (200.1, 122.9)
- removed the H103 at (135.1, 122.9)
- removed the H104 at (264.9, 38.1)
- removed the H104 at (199.8, 38.1)
- removed the H104 at (134.8, 38.1)
- removed the J1 at (244.5, 38.1)
- removed the J1 at (179.5, 38.1)
- removed the J1 at (114.5, 38.1)
- removed the J401 at (221.9, 60.7)
- removed the J401 at (156.9, 60.7)
- removed the J401 at (91.9, 60.7)
- removed the J601 at (248.6, 135.6)
- removed the J601 at (183.6, 135.6)
- removed the J601 at (118.6, 135.6)
- removed the J602 at (227.7, 135.6)
- removed the J602 at (162.7, 135.6)
- removed the J602 at (97.7, 135.6)
- removed the R201 at (246.1, 120.8)
- removed the R201 at (181.1, 120.8)
- removed the R201 at (116.1, 120.8)
- removed the R202 at (237.8, 121.9)
- removed the R202 at (172.8, 121.9)
- removed the R202 at (107.8, 121.9)
- removed the R203 at (246.0, 108.0)
- removed the R203 at (181.0, 108.0)
- removed the R203 at (116.0, 108.0)
- removed the R401 at (229.5, 50.5)
- removed the R401 at (164.5, 50.5)
- removed the R401 at (99.5, 50.5)
- removed the R402 at (229.5, 55.6)
- removed the R402 at (164.5, 55.6)
- removed the R402 at (99.5, 55.6)
- removed the R403 at (229.5, 58.2)
- removed the R403 at (164.5, 58.2)
- removed the R403 at (99.5, 58.2)
- removed the R404 at (228.3, 88.4)
- removed the R404 at (163.3, 88.4)
- removed the R404 at (98.3, 88.4)
- removed the R405 at (228.3, 85.8)
- removed the R405 at (163.3, 85.8)
- removed the R405 at (98.3, 85.8)
- removed the TP201 at (250.0, 101.6)
- removed the TP201 at (185.0, 101.6)
- removed the TP201 at (120.0, 101.6)
- removed the TP202 at (250.0, 104.8)
- removed the TP202 at (185.0, 104.8)
- removed the TP202 at (120.0, 104.8)
- removed the TP203 at (228.9, 112.1)
- removed the TP203 at (163.9, 112.1)
- removed the TP203 at (98.9, 112.1)
- removed the TP204 at (228.9, 108.3)
- removed the TP204 at (163.9, 108.3)
- removed the TP204 at (98.9, 108.3)
- removed the TP205 at (250.0, 108.0)
- removed the TP205 at (185.0, 108.0)
- removed the TP205 at (120.0, 108.0)
- removed the TP206 at (250.0, 98.4)
- removed the TP206 at (185.0, 98.4)
- removed the TP206 at (120.0, 98.4)
- removed the TP207 at (244.1, 118.1)
- removed the TP207 at (179.1, 118.1)
- removed the TP207 at (114.1, 118.1)
- removed the TP208 at (246.7, 114.7)
- removed the TP208 at (181.7, 114.7)
- removed the TP208 at (116.7, 114.7)
- removed the TP209 at (243.3, 89.2)
- removed the TP209 at (178.3, 89.2)
- removed the TP209 at (113.3, 89.2)
- removed the U201 at (237.8, 114.7)
- removed the U201 at (172.8, 114.7)
- removed the U201 at (107.8, 114.7)
- removed the U202 at (237.8, 102.6)
- removed the U202 at (172.8, 102.6)
- removed the U202 at (107.8, 102.6)
- removed the U401 at (234.6, 53.1)
- removed the U401 at (169.6, 53.1)
- removed the U401 at (104.6, 53.1)
- removed the U501 at (257.2, 86.4)
- removed the U501 at (192.2, 86.4)
- removed the U501 at (127.2, 86.4)
- removed the Y201 at (227.0, 102.6)
- removed the Y201 at (162.0, 102.6)
- removed the Y201 at (97.0, 102.6)
- removed the Y401 at (228.3, 78.5)
- removed the Y401 at (163.3, 78.5)
- removed the Y401 at (98.3, 78.5)
Connections:
- U501 pad : GND -> (no net)
Routing:
- net +5V: track 807.1 -> 201.8 mm
- net GND: track 318.1 -> 79.5 mm, vias 56 -> 14
- net /POWER SUPPLY/+18V_IN: track 287.8 -> 71.9 mm
- net /CANBUS CONN/CAN_H: track 202.3 -> 50.6 mm
- net /CANBUS CONN/CAN_L: track 192.7 -> 48.2 mm, vias 8 -> 2
- net /MISO: track 150.9 -> 37.7 mm
- net /SCK: track 142.3 -> 35.6 mm
- net /MOSI: track 131.5 -> 32.9 mm
- net /CANBUS/CS: track 128.6 -> 32.2 mm
- net /MCU/SDA: track 92.5 -> 23.1 mm
- net /CANBUS/INT: track 84.4 -> 21.1 mm
- net /CANBUS/TXCAN: track 61.4 -> 15.4 mm
- net /MCU/SCL: track 60.4 -> 15.1 mm
- net /CANBUS/RXCAN: track 56.5 -> 14.1 mm
- net /POWER SUPPLY/+18V_OUT: track 55.4 -> 13.8 mm
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Other:
- board size 247.1 x 121 mm -> 52.1 x 121 mm

Commit message: sch DRC and THT components position
Parts:
- removed C102: 100nF, Capacitor_SMD:C_0805_2012Metric_Pad1.15x1.40mm_HandSolder
- removed J1: Conn_01x04, Connector_PinHeader_2.54mm:PinHeader_1x04_P2.54mm_Vertical
- added C701: 100nF, Capacitor_SMD:C_0805_2012Metric_Pad1.15x1.40mm_HandSolder, F.Cu at (293.6, -12.4)
- added C702: 100nF, Capacitor_SMD:C_0805_2012Metric_Pad1.15x1.40mm_HandSolder, F.Cu at (222.0, 63.0)
- added C703: 100nF, Capacitor_SMD:C_0805_2012Metric_Pad1.15x1.40mm_HandSolder, F.Cu at (222.0, 60.0)
- added C704: 100nF, Capacitor_SMD:C_0805_2012Metric_Pad1.15x1.40mm_HandSolder, F.Cu at (293.6, -9.42)
- added C705: 10uF, Capacitor_SMD:C_0805_2012Metric_Pad1.15x1.40mm_HandSolder, F.Cu at (230.4, 53.4)
- added C706: 100n, Capacitor_SMD:C_0805_2012Metric_Pad1.15x1.40mm_HandSolder, F.Cu at (347.9, 160.9)
- added C707: 1n, Capacitor_SMD:C_0805_2012Metric_Pad1.15x1.40mm_HandSolder, F.Cu at (350.8, 170.5)
- added C708: 100nF, Capacitor_SMD:C_0805_2012Metric_Pad1.15x1.40mm_HandSolder, F.Cu at (363.0, 183.2)
- added C709: 10u, Capacitor_SMD:C_2512_6332Metric_Pad1.52x3.35mm_HandSolder, F.Cu at (359.0, 185.9)
- added C710: 10u, Capacitor_SMD:C_2512_6332Metric_Pad1.52x3.35mm_HandSolder, F.Cu at (348.8, 177.4)
- added C801: 10uF, Capacitor_SMD:C_0805_2012Metric_Pad1.15x1.40mm_HandSolder, F.Cu at (72.4, 280.7)
- added C802: 100nF, Capacitor_SMD:C_0805_2012Metric_Pad1.15x1.40mm_HandSolder, F.Cu at (77.1, 280.7)
- added C803: 100nF, Capacitor_SMD:C_0805_2012Metric_Pad1.15x1.40mm_HandSolder, F.Cu at (81.9, 280.7)
- added C804: 10uF, Capacitor_SMD:C_0805_2012Metric_Pad1.15x1.40mm_HandSolder, F.Cu at (72.4, 283.6)
- added Cc701: 1uF 100V, Capacitor_SMD:C_1206_3216Metric_Pad1.42x1.75mm_HandSolder, F.Cu at (302.7, -25.2)
- added Cc702: 1uF 100V, Capacitor_SMD:C_1206_3216Metric_Pad1.42x1.75mm_HandSolder, F.Cu at (294.2, -18.8)
- added Cc703: 1uF 100V, Capacitor_SMD:C_1206_3216Metric_Pad1.42x1.75mm_HandSolder, F.Cu at (225.1, 53.6)
- added Cc704: 1uF 100V, Capacitor_SMD:C_1206_3216Metric_Pad1.42x1.75mm_HandSolder, F.Cu at (216.6, 60.1)
- added Cc705: 1uF 100V, Capacitor_SMD:C_1206_3216Metric_Pad1.42x1.75mm_HandSolder, F.Cu at (239.1, 41.3)
- added Cc706: 1uF 100V, Capacitor_SMD:C_1206_3216Metric_Pad1.42x1.75mm_HandSolder, F.Cu at (239.1, 38.0)
- added Cc707: 1uF 100V, Capacitor_SMD:C_1206_3216Metric_Pad1.42x1.75mm_HandSolder, F.Cu at (245.0, 34.7)
- added Cc708: 1uF 100V, Capacitor_SMD:C_1206_3216Metric_Pad1.42x1.75mm_HandSolder, F.Cu at (239.1, 34.7)
- added Cc709: 1uF 100V, Capacitor_SMD:C_1206_3216Metric_Pad1.42x1.75mm_HandSolder, F.Cu at (276.8, 16.1)
- added Cc710: 1uF 100V, Capacitor_SMD:C_1206_3216Metric_Pad1.42x1.75mm_HandSolder, F.Cu at (300.2, -18.8)
- added Cc711: 1uF 100V, Capacitor_SMD:C_1206_3216Metric_Pad1.42x1.75mm_HandSolder, F.Cu at (225.1, 56.9)
- added Cc712: 1uF 100V, Capacitor_SMD:C_1206_3216Metric_Pad1.42x1.75mm_HandSolder, F.Cu at (259.4, 23.8)
- added Ci701: 4,7uF 50V, Capacitor_SMD:C_1206_3216Metric_Pad1.42x1.75mm_HandSolder, F.Cu at (233.4, 47.0)
- added Ci702: 4,7uF 50V, Capacitor_SMD:C_1206_3216Metric_Pad1.42x1.75mm_HandSolder, F.Cu at (259.4, 27.1)
- added Ci703: 4,7uF 50V, Capacitor_SMD:C_1206_3216Metric_Pad1.42x1.75mm_HandSolder, F.Cu at (294.2, -15.5)
- added Co701: 2.2uF 100V, Capacitor_SMD:C_1206_3216Metric_Pad1.42x1.75mm_HandSolder, F.Cu at (300.2, -15.5)
- added Co702: 2.2uF 100V, Capacitor_SMD:C_1206_3216Metric_Pad1.42x1.75mm_HandSolder, F.Cu at (245.0, 38.0)
- added Co703: 2.2uF 100V, Capacitor_SMD:C_1206_3216Metric_Pad1.42x1.75mm_HandSolder, F.Cu at (262.8, 18.9)
- added Co704: 2.2uF 100V, Capacitor_SMD:C_1206_3216Metric_Pad1.42x1.75mm_HandSolder, F.Cu at (268.7, 18.9)
- added Co705: 2.2uF 100V, Capacitor_SMD:C_1206_3216Metric_Pad1.42x1.75mm_HandSolder, F.Cu at (253.4, 30.4)
- added Cs701: 100nF, Capacitor_SMD:C_1206_3216Metric_Pad1.42x1.75mm_HandSolder, F.Cu at (288.3, 4.60)
- added Cs702: 100nF, Capacitor_SMD:C_1206_3216Metric_Pad1.42x1.75mm_HandSolder, F.Cu at (253.4, 27.1)
- added Cs703: 100nF, Capacitor_SMD:C_1206_3216Metric_Pad1.42x1.75mm_HandSolder, F.Cu at (253.4, 23.8)
- added Cs704: 100nF, Capacitor_SMD:C_1206_3216Metric_Pad1.42x1.75mm_HandSolder, F.Cu at (216.6, 63.4)
- added D701: 80CPQ150PbF, KicadZeniteSolarLibrary18:TO-247-3_Horizontal_TabUp, B.Cu at (160.0, 77.5)
- added D702: D_TVS, Diode_SMD:D_0805_2012Metric_Castellated, F.Cu at (347.9, 170.5)
- added D703: D_TVS, Diode_SMD:D_0805_2012Metric_Castellated, F.Cu at (363.0, 188.0)
- added Ds701: BYD77, Diode_SMD:D_MELF_Handsoldering, F.Cu at (215.5, 49.2)
- added Ds702: BYD77, Diode_SMD:D_MELF_Handsoldering, F.Cu at (232.9, 19.4)
- added Ds703: BYD77, Diode_SMD:D_MELF_Handsoldering, F.Cu at (232.9, 23.6)
- added Ds704: BYD77, Diode_SMD:D_MELF_Handsoldering, F.Cu at (244.8, 19.4)
- added F701: Fuse, KicadZeniteSolarLibrary18:Porta_Fusivel, F.Cu at (181.6, 58.4)
- added HS701: Heatsink, KicadZeniteSolarLibrary18:hs10425, B.Cu at (180.3, 33.0)
- added J101: Conn_01x20, Connector_PinHeader_2.54mm:PinHeader_1x20_P2.54mm_Horizontal, F.Cu at (379.7, 166.4)
- added J102: Conn_01x20, Connector_PinSocket_2.54mm:PinSocket_1x20_P2.54mm_Vertical, B.Cu at (127.0, 69.8)
- added J701: Driver_INEP, KicadZeniteSolarLibrary18:Driver_(INEP), B.Cu at (94.0, 31.8)
- added L1/701: L_Core_Iron_Small, KicadZeniteSolarLibrary18:Inductor_Nocoupled, F.Cu at (134.6, 125.7)
- added L2/701: L_Core_Iron_Small, KicadZeniteSolarLibrary18:Inductor_Nocoupled, F.Cu at (177.8, 40.6)
- added L701: L_Small, Inductor_SMD:L_0805_2012Metric_Pad1.15x1.40mm_HandSolder, F.Cu at (217.4, 66.5)
- added MK701: Mounting_Hole, MountingHole:MountingHole_2.2mm_M2_Pad, F.Cu at (253.4, 35.0)
- added Q701: IRFP4321PbF, Package_TO_SOT_THT:TO-247-3_Horizontal_TabUp, B.Cu at (149.9, 67.3)
- added Q702: Q_NPN_Darlington_BEC, Package_TO_SOT_SMD:SOT-23, F.Cu at (357.5, 164.3)
- added R701: 330k, Resistor_SMD:R_0805_2012Metric_Pad1.15x1.40mm_HandSolder, F.Cu at (212.7, 69.4)
- added R702: 330k, Resistor_SMD:R_0805_2012Metric_Pad1.15x1.40mm_HandSolder, F.Cu at (212.7, 66.5)
- added R703: 560k, Resistor_SMD:R_0805_2012Metric_Pad1.15x1.40mm_HandSolder, F.Cu at (244.4, 41.1)
- added R704: 39k, Resistor_SMD:R_0805_2012Metric_Pad1.15x1.40mm_HandSolder, F.Cu at (298.4, -12.4)
- added R705: 10k, Resistor_SMD:R_0805_2012Metric_Pad1.15x1.40mm_HandSolder, F.Cu at (347.9, 165.7)
- added R706: 10k, Resistor_SMD:R_0805_2012Metric_Pad1.15x1.40mm_HandSolder, F.Cu at (359.2, 174.2)
- added R707: 10k, Resistor_SMD:R_0805_2012Metric_Pad1.15x1.40mm_HandSolder, F.Cu at (353.8, 170.5)
- added R708: 8.2k, Resistor_SMD:R_0805_2012Metric_Pad1.15x1.40mm_HandSolder, F.Cu at (362.1, 178.4)
- added R709: 75k, Resistor_SMD:R_0805_2012Metric_Pad1.15x1.40mm_HandSolder, F.Cu at (350.8, 165.8)
- added R710: 15k, Resistor_SMD:R_0805_2012Metric_Pad1.15x1.40mm_HandSolder, F.Cu at (359.2, 179.0)
- added R711: 12k, Resistor_SMD:R_0805_2012Metric_Pad1.15x1.40mm_HandSolder, F.Cu at (356.7, 169.5)
- added R712: 150, Resistor_SMD:R_0805_2012Metric_Pad1.15x1.40mm_HandSolder, F.Cu at (362.1, 173.7)
- added R713: 150, Resistor_SMD:R_0805_2012Metric_Pad1.15x1.40mm_HandSolder, F.Cu at (350.8, 161.0)
- added R714: 100k, Resistor_SMD:R_0805_2012Metric_Pad1.15x1.40mm_HandSolder, F.Cu at (353.8, 164.7)
- added R715: 56k, Resistor_SMD:R_0805_2012Metric_Pad1.15x1.40mm_HandSolder, F.Cu at (359.6, 168.9)
- added R716: 220, Resistor_SMD:R_0805_2012Metric_Pad1.15x1.40mm_HandSolder, F.Cu at (362.6, 168.9)
- added R717: 100, Resistor_SMD:R_0805_2012Metric_Pad1.15x1.40mm_HandSolder, F.Cu at (353.8, 160.0)
- added Rg701: 10k, Resistor_SMD:R_0805_2012Metric_Pad1.15x1.40mm_HandSolder, F.Cu at (305.5, -19.2)
- added Rs701: 100, Resistor_SMD:R_2512_6332Metric_Pad1.52x3.35mm_HandSolder, F.Cu at (231.6, 28.2)
- added Rs702: 100, Resistor_SMD:R_2512_6332Metric_Pad1.52x3.35mm_HandSolder, F.Cu at (231.6, 33.1)
- added Rs703: 100, Resistor_SMD:R_2512_6332Metric_Pad1.52x3.35mm_HandSolder, F.Cu at (225.9, 49.5)
- added Rs704: 100, Resistor_SMD:R_2512_6332Metric_Pad1.52x3.35mm_HandSolder, F.Cu at (231.6, 42.9)
- added Rshunt701: 1500uR, Resistor_SMD:R_2512_6332Metric_Pad1.52x3.35mm_HandSolder, F.Cu at (255.2, 19.7)
- added Rshunt702: 1500uR, Resistor_SMD:R_2512_6332Metric_Pad1.52x3.35mm_HandSolder, F.Cu at (231.6, 38.0)
- added Screw701: +B, MountingHole:MountingHole_5mm_Pad, F.Cu at (198.1, 92.7)
- added Screw702: -B, MountingHole:MountingHole_5mm_Pad, F.Cu at (196.8, 118.1)
- added Screw703: +P, MountingHole:MountingHole_5mm_Pad, F.Cu at (198.1, 71.1)
- added Screw704: -P, MountingHole:MountingHole_5mm_Pad, F.Cu at (199.4, 43.2)
- added TP701: TestPoint_Probe, TestPoint:TestPoint_Pad_D1.0mm, F.Cu at (211.8, 72.4)
- added TP702: TestPoint_Probe, TestPoint:TestPoint_Pad_D1.0mm, F.Cu at (232.0, 50.1)
- added TP703: TestPoint_Probe, TestPoint:TestPoint_Pad_D1.0mm, F.Cu at (307.2, -25.4)
- added TP704: TestPoint_Probe, TestPoint:TestPoint_Pad_D1.0mm, F.Cu at (273.2, 19.3)
- added TP705: TestPoint_Probe, TestPoint:TestPoint_Pad_D1.0mm, F.Cu at (237.9, 44.4)
- added Tvs701: Tvs, Diode_SMD:D_0805_2012Metric_Castellated, F.Cu at (307.0, -22.1)
- added Tvs702: Tvs, Diode_SMD:D_0805_2012Metric_Castellated, F.Cu at (302.2, -22.1)
- added U101: ZCS, KicadZeniteSolarLibrary18:ZCS18, F.Cu at (59.2, 213.4)
- added U102: ZCS, KicadZeniteSolarLibrary18:ZCS18, F.Cu at (129.5, 33.0)
- added U701: INA240A4D, Package_SO:SOIC-8_3.9x4.9mm_P1.27mm, F.Cu at (217.9, 55.2)
- added U702: INA240A4D, Package_SO:SOIC-8_3.9x4.9mm_P1.27mm, F.Cu at (295.5, -23.6)
- added U703: LM324, Package_SO:SOIC-14_3.9x8.7mm_P1.27mm, F.Cu at (351.5, 186.2)
- added U704: INA826, Package_SO:SOIC-8_3.9x4.9mm_P1.27mm, F.Cu at (354.5, 177.1)
- added U801: LM7812_TO220, KicadZeniteSolarLibrary18:TO-220-3_Horizontal_TabDown_SMD, F.Cu at (61.7, 299.4)
- moved C402 305.0 mm to (-266.4, 27.7)
- moved D401 305.0 mm to (-272.2, 7.62)
- moved J602 305.0 mm to (-269.5, 95.0)
- moved U401 305.0 mm to (-262.6, 12.4)
- moved C201 305.0 mm to (-262.3, 53.3)
- moved C202 305.0 mm to (-254.6, 69.2)
- moved C203 305.0 mm to (-269.9, 59.4)
- moved C204 305.0 mm to (-267.7, 55.6)
- moved C205 305.0 mm to (-259.5, 79.1)
- moved C401 305.0 mm to (-251.2, 32.8)
- moved C403 305.0 mm to (-269.0, 35.3)
- moved C404 305.0 mm to (-267.7, 30.9)
- moved C405 305.0 mm to (-267.7, 12.4)
- moved C406 305.0 mm to (-265.3, 7.49)
- moved C501 305.0 mm to (-239.2, 55.2)
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Connections:
- net /POWER SUPPLY/+18V_OUT renamed VCC
- U401 pad 16: Net-(U401-Pad16) -> /MCU/PWM
- U401 pad 23: Net-(U401-Pad23) -> /MCU/V_Vpanel_ADC
- U401 pad 24: Net-(U401-Pad24) -> /MCU/V_Ipanel_ADC
- U401 pad 25: Net-(U401-Pad25) -> /MCU/V_Vbat_ADC
- U401 pad 26: Net-(U401-Pad26) -> /MCU/V_Ibat_ADC
- U401 pad 27: /MCU/SDA -> Net-(U401-Pad27)
- U401 pad 28: /MCU/SCL -> Net-(U401-Pad28)
Routing:
- net /MCU/SDA: track 23.1 -> 0.00 mm
- net Net-(U401-Pad27): track 0.00 -> 23.1 mm
- net Net-(U401-Pad28): track 0.00 -> 15.1 mm
- net /MCU/SCL: track 15.1 -> 0.00 mm
Other:
- board outline removed

Commit message: parte de potencia
Parts:
- D701, Q701: moved to F.Cu
- Rshunt701, Rshunt702: footprint Resistor_SMD:R_2512_6332Metric_Pad1.52x3.35mm_HandSolder -> KicadZeniteSolarLibrary18:PML100HZPJV0L5
- moved C201 260.8 mm to (-63.5, 222.2)
- moved C202 260.8 mm to (-55.9, 238.1)
- moved C203 260.8 mm to (-71.1, 228.3)
- moved C204 260.8 mm to (-69.0, 224.5)
- moved C205 260.8 mm to (-60.7, 248.0)
- moved C401 260.8 mm to (-52.5, 201.7)
- moved C402 260.8 mm to (-67.7, 196.6)
- moved C403 260.8 mm to (-70.2, 204.2)
- moved C404 260.8 mm to (-69.0, 199.8)
- moved C405 260.8 mm to (-69.0, 181.4)
- moved C406 260.8 mm to (-66.5, 176.4)
- moved C501 260.8 mm to (-40.4, 224.2)
- moved C502 260.8 mm to (-40.4, 220.3)
- moved C503 260.8 mm to (-47.0, 223.5)
- moved C504 260.8 mm to (-47.0, 220.3)
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Connections:
- net Net-(F701-Pad2) renamed /Sheet5F261196/-P_unfused
- L1/701 pad 1: /Sheet5F261196/HS -> /Sheet5F261196/+B
- L1/701 pad 2: /Sheet5F261196/+B -> /Sheet5F261196/HS
- L2/701 pad 1: /Sheet5F261196/-Vp -> /Sheet5F261196/HS
- L2/701 pad 2: /Sheet5F261196/HS -> /Sheet5F261196/-Vp
Routing:
- net /Sheet5F261196/-B: track 0.00 -> 109.8 mm
- net /Sheet5F261196/+Vp: track 0.00 -> 103.4 mm
- net /Sheet5F261196/+B: track 0.00 -> 73.9 mm
- net /Sheet5F261196/-Vp: track 0.00 -> 45.0 mm
- net /Sheet5F261196/HS: track 0.00 -> 40.8 mm
- net /Sheet5F261196/BatShunt+: track 0.00 -> 27.9 mm
- net /Sheet5F261196/PanelShunt-: track 0.00 -> 8.27 mm
- added copper zone on F.Cu, net (none)
- added copper zone on F.Cu, net /Sheet5F261196/+B

Commit message: initial
Parts:
- moved H101 299.7 mm to (224.2, 163.8), turned to 180 degrees
- moved D501 299.1 mm to (246.4, 135.9), turned to 0 degrees
- moved TP206 294.4 mm to (235.6, 149.5), turned to 0 degrees
- moved C503 289.4 mm to (232.4, 148.0), turned to 90 degrees
- moved F501 287.8 mm to (237.5, 135.9), turned to 180 degrees
- moved C501 285.7 mm to (233.0, 141.4), turned to 270 degrees
- moved C504 285.5 mm to (229.2, 147.9), turned to 90 degrees
- moved C502 281.0 mm to (229.2, 141.4), turned to 270 degrees
- moved H103 276.3 mm to (214.0, 128.3), turned to 0 degrees
- moved U501 274.5 mm to (223.5, 142.2), turned to 270 degrees
- moved J602 267.8 mm to (187.1, 191.4), turned to 90 degrees
- moved H104 260.8 mm to (224.2, 205.7), turned to 180 degrees
- moved H102 256.7 mm to (174.4, 197.2), turned to 0 degrees
- moved J601 254.7 mm to (187.1, 170.6), turned to 90 degrees
- moved R202 244.0 mm to (173.4, 181.4), turned to 270 degrees
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Routing:
- net /MISO: track 37.7 -> 16.0 mm
- net /Sheet5F261196/+B: track 73.9 -> 54.1 mm
- net /MOSI: track 32.9 -> 13.4 mm
- net /Sheet5F261196/BatShunt+: track 27.9 -> 9.24 mm
- net /Sheet5F261196/+Vp: track 103.4 -> 86.5 mm
- net /POWER SUPPLY/+18V_IN: track 71.9 -> 56.2 mm
- net /CANBUS/CS: track 32.2 -> 18.9 mm
- net /SCK: track 35.6 -> 23.3 mm
- net /CANBUS/INT: track 21.1 -> 10.8 mm
- net +5V: track 201.8 -> 194.6 mm
- removed copper zone on B.Cu, net GND
