File: hardware/MCC20.kicad_pcb (KiCad board)
At the start: 2 copper layers, 149 parts, among them J101 Conn_01x20, J102 Conn_01x20, J401 USART, J601 RJ45, J602 RJ45, J701 Driver_INEP, Q701 IRFP4321PbF, Q702 Q_NPN_Darlington_BEC, U101 ZCS, U102 ZCS, U201 MCP2551-I/SN, U202 MCP2515-xSO, U401 ATMEGA328P-PU, U501 LM7805, U701 INA240A4D, U702 INA240A4D, U703 LM324, U704 INA826, U801 LM7812_TO220, Y201 16MHz, Y401 16MHz

Commit message: snubber
Parts:
- C701, C702, C703, C704, C705, Cs701, Cs702, Cs703, Cs704, Ds701, Ds702, Ds703, Ds704, L1/701, L2/701, L701, R701, R702, R703, R704, Rg701, Rs701, Rs702, Rs703, Rs704, TP701, TP702, TP703, TP704, TP705, Tvs701, Tvs702: moved to B.Cu
- HS701: moved to F.Cu
- J102: footprint Connector_PinSocket_2.54mm:PinSocket_1x20_P2.54mm_Vertical -> Connector_PinSocket_2.54mm:PinSocket_1x20_P2.54mm_Vertical_SMD_Pin1Left
- J701: footprint KicadZeniteSolarLibrary18:Driver_(INEP) -> KicadZeniteSolarLibrary18:Driver_(INEP)_SMD
- moved D403 204.0 mm to (84.1, 85.2)
- moved J601 204.0 mm to (108.2, 135.0)
- moved R405 204.0 mm to (87.9, 85.2)
- moved C201 204.0 mm to (94.6, 93.3)
- moved C202 204.0 mm to (102.2, 109.2)
- moved C203 204.0 mm to (87.0, 99.4)
- moved C204 204.0 mm to (89.2, 95.6)
- moved C205 204.0 mm to (97.4, 119.1)
- moved C402 204.0 mm to (90.4, 67.7)
- moved C403 204.0 mm to (87.9, 75.3)
- moved C405 204.0 mm to (89.2, 52.5)
- moved C406 204.0 mm to (91.6, 47.5)
- moved D201 204.0 mm to (105.7, 124.2)
- moved D401 204.0 mm to (84.6, 47.6)
- moved D402 204.0 mm to (84.1, 87.7)
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Connections:
- L1/701 pad 1: /Sheet5F261196/+B -> /Sheet5F261196/HS
- L1/701 pad 2: /Sheet5F261196/HS -> /Sheet5F261196/+B
- L2/701 pad 1: /Sheet5F261196/HS -> /Sheet5F261196/-Vp
- L2/701 pad 2: /Sheet5F261196/-Vp -> /Sheet5F261196/HS
Routing:
- net /Sheet5F261196/+Vp: track 103.4 -> 146.5 mm
- net /Sheet5F261196/HS: track 40.8 -> 83.7 mm
- net +5V: track 201.8 -> 162.1 mm
- net Net-(Cs702-Pad2): track 0.00 -> 27.6 mm
- net /POWER SUPPLY/+18V_IN: track 71.9 -> 47.0 mm
- net Net-(U401-Pad27): track 23.1 -> 0.00 mm
- net Net-(Cs703-Pad2): track 0.00 -> 21.2 mm
- net /Sheet5F261196/HG: track 0.00 -> 18.6 mm
- net Net-(U401-Pad28): track 15.1 -> 0.36 mm
- net /Sheet5F261196/-B: track 109.8 -> 123.2 mm
- net /Sheet5F261196/BatShunt+: track 27.9 -> 21.7 mm
- net Net-(Cs701-Pad2): track 0.00 -> 5.32 mm
- net Net-(Cs704-Pad1): track 0.00 -> 4.54 mm
- net VCC: track 13.8 -> 9.68 mm
- net GND: track 79.5 -> 75.7 mm, vias 14 -> 12
